File: pcb/pcb.kicad_sch (KiCad schematic)
At the start: 49 parts, among them J1 MJ-4PP-9, SW1 SW_PUSH, SW10 SW_PUSH, SW11 SW_PUSH, SW12 SW_PUSH, SW13 SW_PUSH, SW14 SW_PUSH, SW15 SW_PUSH, SW16 SW_PUSH, SW17 SW_PUSH, SW18 SW_PUSH, SW2 SW_PUSH, SW3 SW_PUSH, SW4 SW_PUSH, SW5 SW_PUSH, SW6 SW_PUSH, SW7 SW_PUSH, SW8 SW_PUSH, SW9 SW_PUSH, U1 xiao-ble, U2 xiao-ble

Commit message: improve pcb
Parts:
- added BATTCONN2, BATTCONN3: Conn_01x02_Female, picachoc:JST_PH_S2B-PH-K_1x02_P2.00mm, symbol Connector:Conn_01x02_Female
Connections:
- net BATT: now also BATTCONN2.1 (Pin_1), BATTCONN3.1 (Pin_1)
- net GND: now also BATTCONN2.2 (Pin_2), BATTCONN3.2 (Pin_2)
- net SW_ENCA: now also RE1.S2; no longer RE1.S1
- net SW_ENCB: now also RE1.S1; no longer RE1.S2
Changed lines of the file:
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@@
+    )
+  )
+  (global_label "BATT" (shape input) (at 238.76 140.97 180) (fields_autoplaced)
+    (effects (font (size 1.27 1.27)) (justify right))
+    (property "Intersheet References" "${INTERSHEET_REFS}" (id 0) (at 232.0531 140.8906 0)
+      (effects (font (size 1.27 1.27)) (justify right) hide)
     )
   )
@@
     )
   )
-  (global_label "SW_ENCA" (shape input) (at 195.58 129.54 0) (fields_autoplaced)
-    (effects (font (size 1.27 1.27)) (justify left))
-    (property "Intersheet References" "${INTERSHEET_REFS}" (id 0) (at 206.4598 129.4606 0)
+  (global_label "SW_ENCA" (shape input) (at 195.58 134.62 0) (fields_autoplaced)
+    (effects (font (size 1.27 1.27)) (justify left))
+    (property "Intersheet References" "${INTERSHEET_REFS}" (id 0) (at 206.4598 134.5406 0)
       (effects (font (size 1.27 1.27)) (justify left) hide)
     )
@@
     )
   )
-  (global_label "SW_ENCB" (shape input) (at 195.58 134.62 0) (fields_autoplaced)
-    (effects (font (size 1.27 1.27)) (justify left))
-    (property "Intersheet References" "${INTERSHEET_REFS}" (id 0) (at 206.6412 134.5406 0)
+  (global_label "BATT" (shape input) (at 238.76 154.94 180) (fields_autoplaced)
+    (effects (font (size 1.27 1.27)) (justify right))
+    (property "Intersheet References" "${INTERSHEET_REFS}" (id 0) (at 232.0531 154.8606 0)
+      (effects (font (size 1.27 1.27)) (justify right) hide)
+    )
+  )
+  (global_label "SW_ENCB" (shape input) (at 195.58 129.54 0) (fields_autoplaced)
+    (effects (font (size 1.27 1.27)) (justify left))
+    (property "Intersheet References" "${INTERSHEET_REFS}" (id 0) (at 206.6412 129.4606 0)
       (effects (font (size 1.27 1.27)) (justify left) hide)
     )
@@
     (pin "1")
   )
+  (symbol (lib_id "power:GND") (at 238.76 157.48 0) (unit 1)
+    (in_bom yes) (on_board yes) (fields_autoplaced)
+    (property "Reference" "#PWR01" (id 0) (at 238.76 163.83 0)
+      (effects (font (size 1.27 1.27)) hide)
+    )
+    (property "Value" "GND" (id 1) (at 238.76 162.56 0))
+    (property "Footprint" "" (id 2) (at 238.76 157.48 0)
+      (effects (font (size 1.27 1.27)) hide)
+    )
+    (property "Datasheet" "" (id 3) (at 238.76 157.48 0)
+      (effects (font (size 1.27 1.27)) hide)
+    )
+    (pin "1")
+  )
   (symbol (lib_id "power:GND") (at 80.01 27.94 0) (mirror y) (unit 1)
     (in_bom yes) (on_board yes)
@@
     )
     (pin "1")
+  )
+  (symbol (lib_id "Connector:Conn_01x02_Female") (at 243.84 154.94 0) (unit 1)
+    (in_bom yes) (on_board yes) (fields_autoplaced)
+    (property "Reference" "BATTCONN3" (id 0) (at 245.11 154.9399 0)
+      (effects (font (size 1.27 1.27)) (justify left))
+    )
+    (property "Value" "Conn_01x02_Female" (id 1) (at 245.11 157.4799 0)
+      (effects (font (size 1.27 1.27)) (justify left))
+    )
+    (property "Footprint" "picachoc:JST_PH_S2B-PH-K_1x02_P2.00mm" (id 2) (at 243.84 154.94 0)
+      (effects (font (size 1.27 1.27)) hide)
+    )
+    (property "Datasheet" "~" (id 3) (at 243.84 154.94 0)
+      (effects (font (size 1.27 1.27)) hide)
+    )
+    (pin "1")
+    (pin "2")
   )
   (symbol (lib_id "typec:HRO-TYPE-C-31-M-12") (at 264.16 39.37 0) (unit 1)
@@
     (pin "2")
   )
+  (symbol (lib_id "Connector:Conn_01x02_Female") (at 243.84 140.97 0) (unit 1)
+    (in_bom yes) (on_board yes) (fields_autoplaced)
+    (property "Reference" "BATTCONN2" (id 0) (at 245.11 140.9699 0)
+      (effects (font (size 1.27 1.27)) (justify left))
+    )
+    (property "Value" "Conn_01x02_Female" (id 1) (at 245.11 143.5099 0)
+      (effects (font (size 1.27 1.27)) (justify left))
+    )
+    (property "Footprint" "picachoc:JST_PH_S2B-PH-K_1x02_P2.00mm" (id 2) (at 243.84 140.97 0)
+      (effects (font (size 1.27 1.27)) hide)
+    )
+    (property "Datasheet" "~" (id 3) (at 243.84 140.97 0)
+      (effects (font (size 1.27 1.27)) hide)
+    )
+    (pin "1")
+    (pin "2")
+  )
   (symbol (lib_id "power:VCC") (at 110.49 24.13 0) (unit 1)
     (in_bom yes) (on_board yes)
@@
     (pin "1")
     (pin "2")
+  )
+  (symbol (lib_id "power:GND") (at 238.76 143.51 0) (unit 1)
+    (in_bom yes) (on_board yes) (fields_autoplaced)
+    (property "Reference" "#PWR0101" (id 0) (at 238.76 149.86 0)
+      (effects (font (size 1.27 1.27)) hide)
+    )
+    (property "Value" "GND" (id 1) (at 238.76 148.59 0))
+    (property "Footprint" "" (id 2) (at 238.76 143.51 0)
+      (effects (font (size 1.27 1.27)) hide)
+    )
+    (property "Datasheet" "" (id 3) (at 238.76 143.51 0)
+      (effects (font (size 1.27 1.27)) hide)
+    )
+    (pin "1")
   )
   (symbol (lib_id "kbd:SW_PUSH") (at 81.28 113.03 0) (unit 1)
@@
       (reference "#FLG02") (unit 1) (value "PWR_FLAG") (footprint "")
     )
+    (path "/24a83dc0-56f7-441f-9cd2-63988ea40d6d"
+      (reference "#PWR01") (unit 1) (value "GND") (footprint "")
+    )
     (path "/83a9da6c-4adb-4040-b241-3f7492a2322f"
       (reference "#PWR02") (unit 1) (value "GND") (footprint "")
@@
       (reference "#PWR023") (unit 1) (value "GND") (footprint "")
     )
+    (path "/e8dba17b-4455-4c3b-bffa-1cef7698efac"
+      (reference "#PWR0101") (unit 1) (value "GND") (footprint "")
+    )
     (path "/5148de54-ef71-4b99-9090-275a7c3d70ab"
       (reference "BATTCONN1") (unit 1) (value "Conn_01x02_Female") (footprint "picachoc:JST_PH_S2B-PH-K_1x02_P2.00mm")
     )
+    (path "/d31eb9c7-33a2-4357-bd65-c2e4560d2073"
+      (reference "BATTCONN2") (unit 1) (value "Conn_01x02_Female") (footprint "picachoc:JST_PH_S2B-PH-K_1x02_P2.00mm")
+    )
+    (path "/915e0225-ec43-4fca-ba3d-3d6b6935d9fd"
+      (reference "BATTCONN3") (unit 1) (value "Conn_01x02_Female") (footprint "picachoc:JST_PH_S2B-PH-K_1x02_P2.00mm")
+    )
     (path "/f48246bb-eadf-4a25-81a4-925b403a988f"

Commit message: small pcb
Parts:
- removed BATTCONN1, BATTCONN2, BATTCONN3: Conn_01x02_Female, picachoc:JST_PH_S2B-PH-K_1x02_P2.00mm, symbol Connector:Conn_01x02_Female
- removed BATTSW1, BATTSW2: SW_SPDT, Button_Switch_SMD:SW_SPDT_PCM12, symbol Switch:SW_SPDT
- removed JP1, JP2, JP3: SolderJumper_2_Open, Jumper:SolderJumper-2_P1.3mm_Open_TrianglePad1.0x1.5mm, symbol Jumper:SolderJumper_2_Open
- removed U1, U2: xiao-ble, picachoc:xiao-ble-smd, symbol kleeb-mcu:xiao-ble
- removed USB1, USB2: HRO-TYPE-C-31-M-12, picachoc:HRO-TYPE-C-31-M-12-data, symbol typec:HRO-TYPE-C-31-M-12
- added H1, H2, H3, H4: MountingHole, picachoc:spacer_m2_3.4, symbol Mechanical:MountingHole
- added H5, H6: MountingHole, kbd:thread_m2, symbol Mechanical:MountingHole
- added J2, J3: Conn_01x12_Female, Connector_FFC-FPC:TE_1-1734839-2_1x12-1MP_P0.5mm_Horizontal, symbol Connector:Conn_01x12_Female
- added J4: Conn_01x05_Female, Connector_PinHeader_2.54mm:PinHeader_1x05_P2.54mm_Vertical, symbol Connector:Conn_01x05_Female
- added U1, U2: rp2040-zero, picachoc:rp2040-zero-smd, symbol kleeb-mcu:rp2040-zero
- SW1, SW10, SW11, SW12, SW13, SW14, SW15, SW16, SW17, SW18, SW2, SW3, SW4, SW5, SW6, SW7, SW8, SW9: footprint picachoc:Kailh-PG1350-1u -> picachoc:Kailh_PG1350_hotswap
Connections:
- net ENCA: now also U1.15 (14), U2.15 (14)
- net ENCB: now also U1.9 (8), U2.9 (8); no longer J1.B
- net GND: now also J2.2 (Pin_2), J3.2 (Pin_2), J4.4 (Pin_4), U1.22 (GND), U2.22 (GND)
- net VCC: now also J2.1 (Pin_1), J3.1 (Pin_1), J4.3 (Pin_3), U1.21 (3V3), U2.21 (3V3)
- net col0: now also U1.20 (29), U2.20 (29)
- net col1: now also U1.19 (28), U2.19 (28)
- net col2: now also U1.18 (27), U2.18 (27)
- net col3: now also U1.17 (26), U2.17 (26)
- net row0: now also U1.10 (9), U2.10 (9)
- net row1: now also U1.11 (10), U2.11 (10)
- net row2: now also U1.13 (12), U2.13 (12)
- net row3: now also U1.14 (13), U2.14 (13)
- net DATA renamed TX
- net TX: now also U1.1 (0), U2.1 (0)
- net SW_ENCB renamed col4
- net col4: now also U1.16 (15), U2.16 (15)
- new net CS: J2.10 (Pin_10), J3.10 (Pin_10), J4.5 (Pin_5), U1.6 (5), U2.6 (5)
- new net MISO: J2.11 (Pin_11), J3.11 (Pin_11), U1.5 (4), U2.5 (4)
- new net MOSI: J2.8 (Pin_8), J3.8 (Pin_8), J4.1 (Pin_1), U1.4 (3), U2.4 (3)
- new net RX: J1.B, U1.2 (1), U2.2 (1)
- new net SCK: J2.12 (Pin_12), J3.12 (Pin_12), J4.2 (Pin_2), U1.3 (2), U2.3 (2)
- no-connect marks 26 -> 20
Other:
- moved on the sheet: D1, D10, D11, D12, D13, D14, D15, D16, D17, D18, D19, D2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

Commit message: new version
Parts:
- removed H5, H6: MountingHole, kbd:thread_m2, symbol Mechanical:MountingHole
- removed J2, J3: Conn_01x12_Female, Connector_FFC-FPC:TE_1-1734839-2_1x12-1MP_P0.5mm_Horizontal, symbol Connector:Conn_01x12_Female
- removed J4: Conn_01x05_Female, Connector_PinHeader_2.54mm:PinHeader_1x05_P2.54mm_Vertical, symbol Connector:Conn_01x05_Female
- added J2: USB_C_Receptacle_USB2.0, zzkeeb:Connector_USB-C-mid-mount-ali-reversible-data, symbol Connector:USB_C_Receptacle_USB2.0
- added LED1, LED10, LED11, LED12, LED13, LED14, LED15, LED16, LED17, LED18, LED2, LED3, LED4, LED5, LED6, LED7, LED8, LED9: YS-SK6812MINI-E, zzkeeb:LED_SK6812-MINI-E-reversible, symbol kbd:YS-SK6812MINI-E
- added U3: roller, zzkeeb:RotaryEncoder_EVQWGD001, symbol zzkeeb:RollerEncoder_EVQWGD001
- D1, D10, D11, D12, D13, D14, D15, D16, D17, D18, D19, D2, D3, D4, D5, D6, D7, D8, D9: footprint picachoc:D3_SMD -> zzkeeb:Diode_1N4148-SOD123-reversible
- H1, H2, H3, H4: footprint picachoc:spacer_m2_3.4 -> zzkeeb:Hole_M2-spacer
- J1: footprint picachoc:MJ-4PP-9 -> zzkeeb:Connector_TRRS-reversible
- RE1: footprint picachoc:RotaryEncoder_EC11 -> zzkeeb:RotaryEncoder_EC11
- SW1, SW10, SW11, SW12, SW13, SW14, SW15, SW16, SW17, SW18, SW2, SW3, SW4, SW5, SW6, SW7, SW8, SW9: footprint picachoc:Kailh_PG1350_hotswap -> zzkeeb:Switch_ChocV1-hotswap-reversible
- U1, U2: footprint picachoc:rp2040-zero-smd -> zzkeeb:MCU_rp2040-zero-smd
Connections:
- net ENCA: now also U1.17 (26), U2.7 (6), U3.A; no longer U1.15 (14), U2.15 (14)
- net ENCB: now also U1.7 (6), U2.17 (26), U3.B; no longer U1.9 (8), U2.9 (8)
- net GND: now also J2.A1 (GND), J2.A12 (GND), J2.B1 (GND), J2.B12 (GND), LED1.3 (VSS), LED10.3 (VSS), LED11.3 (VSS), LED12.3 (VSS), LED13.3 (VSS), LED14.3 (VSS), LED15.3 (VSS), LED16.3 (VSS), LED17.3 (VSS), LED18.3 (VSS), LED2.3 (VSS), LED3.3 (VSS), LED4.3 (VSS), LED5.3 (VSS), LED6.3 (VSS), LED7.3 (VSS), LED8.3 (VSS), LED9.3 (VSS), U3.C
- net RX: now also J2.A6 (D+), J2.B6 (D+)
- net SW_ENCA: now also D16.2 (A), U3.S2; no longer D19.2 (A)
- net TX: now also J2.A7 (D-), J2.B7 (D-)
- net VCC: now also J2.A4 (VBUS), J2.A9 (VBUS), J2.B4 (VBUS), J2.B9 (VBUS), LED1.1 (VDD), LED10.1 (VDD), LED11.1 (VDD), LED12.1 (VDD), LED13.1 (VDD), LED14.1 (VDD), LED15.1 (VDD), LED16.1 (VDD), LED17.1 (VDD), LED18.1 (VDD), LED2.1 (VDD), LED3.1 (VDD), LED4.1 (VDD), LED5.1 (VDD), LED6.1 (VDD), LED7.1 (VDD), LED8.1 (VDD), LED9.1 (VDD)
- net col0: now also SW10.2, SW15.2, SW5.2, U1.10 (9), U2.14 (13); no longer SW1.2, SW11.2, SW6.2, U1.20 (29), U2.20 (29)
- net col1: now also RE1.S1, SW1.2, SW11.2, SW6.2, U1.11 (10), U2.13 (12), U3.S1; no longer SW12.2, SW16.2, SW2.2, SW7.2, U1.19 (28), U2.19 (28)
- net col2: now also SW12.2, SW16.2, SW2.2, SW7.2, U1.12 (11), U2.12 (11); no longer SW13.2, SW17.2, SW3.2, SW8.2, U1.18 (27), U2.18 (27)
- net col3: now also SW13.2, SW17.2, SW3.2, SW8.2, U1.13 (12), U2.11 (10); no longer SW14.2, SW18.2, SW4.2, SW9.2, U1.17 (26), U2.17 (26)
- net col4: now also SW14.2, SW18.2, SW4.2, SW9.2, U1.14 (13), U2.10 (9); no longer RE1.S1, SW10.2, SW15.2, SW5.2, U1.16 (15), U2.16 (15)
- net row0: now also U1.16 (15), U2.8 (7); no longer D5.1 (K), U1.10 (9), U2.10 (9)
- net row1: now also D5.1 (K), U1.15 (14), U2.9 (8); no longer D10.1 (K), U1.11 (10), U2.11 (10)
- net row2: now also D10.1 (K), U1.9 (8), U2.15 (14); no longer D15.1 (K), U1.13 (12), U2.13 (12)
- net row3: now also D15.1 (K), U1.8 (7), U2.16 (15); no longer U1.14 (13), U2.14 (13)
- net at SW17.1: now also D18.2 (A); no longer D17.2 (A)
- net at SW16.1: now also D17.2 (A); no longer D16.2 (A)
- net at SW18.1: now also D19.2 (A); no longer D18.2 (A)
- net CS: no longer names the net of U1.6 (5)
- net CS: no longer U2.6 (5)
- net MISO: no longer names the net of U1.5 (4)
- net MISO: no longer U2.5 (4)
- net MOSI: no longer names the net of U1.4 (3)
- net MOSI: no longer U2.4 (3)
- net SCK: no longer names the net of U1.3 (2)
- net SCK: no longer U2.3 (2)
- new net: LED2.2 (DOUT), LED3.4 (DIN)
- new net: LED1.2 (DOUT), LED2.4 (DIN)
- new net: LED10.2 (DOUT), LED11.4 (DIN)
- new net: LED10.4 (DIN), LED5.2 (DOUT)
- new net: LED12.2 (DOUT), LED13.4 (DIN)
- new net: LED11.2 (DOUT), LED12.4 (DIN)
- new net: LED8.4 (DIN), LED9.2 (DOUT)
- new net: LED4.2 (DOUT), LED9.4 (DIN)
- new net: LED17.4 (DIN), LED18.2 (DOUT)
- new net: LED14.2 (DOUT), LED18.4 (DIN)
- new net: LED13.2 (DOUT), LED14.4 (DIN)
- new net: LED3.2 (DOUT), LED4.4 (DIN)
- new net: LED16.4 (DIN), LED17.2 (DOUT)
- new net: LED5.4 (DIN), LED6.2 (DOUT)
- new net: LED7.4 (DIN), LED8.2 (DOUT)
- new net: LED15.4 (DIN), LED16.2 (DOUT)
- new net: LED6.4 (DIN), LED7.2 (DOUT)
- new net LED: LED1.4 (DIN), U1.19 (28), U2.19 (28)
- no-connect marks 20 -> 21
Other:
- moved on the sheet: J1, RE1
